Commit message: remove the mimic elements

File: src/my_project/robot.urdf (robot description, URDF)
Before this commit: robot panda, 12 links, 11 joints
Joints:
- joint panda_finger_joint2: mimic joint=panda_finger_joint1 -> (none)

File: src/robots/hand.xacro (robot description, xacro)
@@ -96,5 +96,4 @@
       <axis xyz="0 -1 0"/>
       <limit effort="20" lower="0.0" upper="0.04" velocity="0.2"/>
-      <mimic joint="${ns}_finger_joint1" />
     </joint>
   </xacro:macro>
